Commit message: Gazebo world building, camera inputs, camera points

File: dev/src/sample_robo/description/example_gazebo.xacro (robot description, xacro)
@@ -55,4 +55,5 @@
             try swapping "depth" to "camera"-->
     <gazebo reference="camera_link">
+        <!-- <sensor type="camera" name="my_camera"> -->
         <sensor type="depth" name="my_camera">
             <update_rate>20</update_rate>

File: dev/src/sample_robo/description/example_robot.urdf.xacro (robot description, xacro)
@@ -84,4 +84,5 @@
         <axis xyz="0 -1 0"/>
         <limit lower="0" upper="${pi/2}" velocity="100" effort="100"/>
+        <dynamics damping="10.0" friction="10.0"/>
     </joint>
     <!-- arm_link describes the arm -->
